File: Electrical_Schematics/Schematic_v1/Schematic_v1.kicad_sch (KiCad schematic)
At the start: 0 parts

Commit message: finish schematic
Parts:
- added BT1: Battery, symbol Device:Battery
- added LS1: Speaker, symbol Device:Speaker
- added U1: (no value), symbol Custom Board:ESP32-S3-WROOM-1-N16R8
- added U2: MAX98357A, Package_DFN_QFN:TQFN-16-1EP_3x3mm_P0.5mm_EP1.23x1.23mm, symbol Audio:MAX98357A
- added U3: (no value), symbol Custom Board:Unnamed_battery_charge-and-boost_module
Connections:
- new net: BT1.1 (+), U3. (BAT-)
- new net: BT1.2 (-), U3. (BAT-)
- new net: U1.5 (IO5), U2.16 (BCLK)
- new net: U1.6 (IO6), U2.14 (LRCLK)
- new net: U1.7 (IO7), U2.1 (DIN)
- new net: LS1.1, U2.9 (OUTP)
- new net: LS1.2, U2.10 (OUTN)
- new net +5V: U2.7 (VDD), U2.8 (VDD), U3. (BAT-)
- new net GND: U1.23 (GND), U2.11 (GND), U2.15 (GND), U2.3 (GND), U3. (BAT-)
Other:
- title: (none) -> Dog Communication Device
